Commit message: Add reverse paramter for link2.

File: open_manipulator_x_description/urdf/open_manipulator_x.xacro (robot description, xacro)
@@ -3,5 +3,5 @@
 <!-- Import Rviz colors -->
 <xacro:include filename="$(find open_manipulator_x_description)/urdf/open_manipulator_x.material.xacro" />
-<xacro:macro name="open_manipulator_x" params="parent *origin">
+<xacro:macro name="open_manipulator_x" params="parent link2_reversed:='false' *origin">
   <joint name="origin_to_link1" type="fixed">
     <xacro:insert_block name="origin" />
@@ -36,6 +36,11 @@
   <joint name="joint1" type="revolute">
     <parent link="link1"/>
-    <child link="link2"/>
-    <origin xyz="0.012 0.0 0.017" rpy="0 0 0"/>
+	<child link="link2"/>
+	<xacro:unless value="${link2_reversed}" >
+		<origin xyz="0.012 0.0 0.017" rpy="0 0 0"/>
+	</xacro:unless>
+	<xacro:if value="${link2_reversed}" >
+		<origin xyz="0.012 0.0 0.017" rpy="0 0 3.1415"/>
+	</xacro:if>
     <axis xyz="0 0 1"/>
     <limit velocity="4.8" effort="1" lower="-2.82743338823" upper="2.82743338823" />
